Commit message: add URDF

File: megabot/robot.urdf (robot description, URDF)
Before this commit: robot megabot, 77 links, 76 joints
Links:
- removed link chassis
- removed link connecteur
- removed link connecteur_10
- removed link connecteur_11
- removed link connecteur_12
- removed link connecteur_13
- removed link connecteur_14
- removed link connecteur_15
- removed link connecteur_16
- removed link connecteur_17
- removed link connecteur_18
- removed link connecteur_19
- removed link connecteur_2
- removed link connecteur_20
- removed link connecteur_21
- removed link connecteur_22
- removed link connecteur_23
- removed link connecteur_24
- removed link connecteur_25
- removed link connecteur_26
- removed link connecteur_27
- removed link connecteur_28
- removed link connecteur_29
- removed link connecteur_3
- removed link connecteur_30
- removed link connecteur_31
- removed link connecteur_32
- removed link connecteur_4
- removed link connecteur_5
- removed link connecteur_6
- removed link connecteur_7
- removed link connecteur_8
- removed link connecteur_9
- removed link cuisse
- removed link cuisse_2
- removed link cuisse_3
- removed link cuisse_4
- removed link hanche
- removed link hanche_2
- removed link hanche_3
- removed link hanche_4
- removed link pied
- removed link pied_2
- removed link pied_3
- removed link pied_4
- removed link support_v2
- removed link support_v2_2
- removed link support_v2_3
- removed link support_v2_4
- removed link vérin_f
- removed link vérin_f_10
- removed link vérin_f_11
- removed link vérin_f_12
- removed link vérin_f_2
- removed link vérin_f_3
- removed link vérin_f_4
- removed link vérin_f_5
- removed link vérin_f_6
- removed link vérin_f_7
- removed link vérin_f_8
- removed link vérin_f_9
- removed link vérin_m
- removed link vérin_m_10
- removed link vérin_m_11
- removed link vérin_m_12
- removed link vérin_m_2
- removed link vérin_m_3
- removed link vérin_m_4
- removed link vérin_m_5
- removed link vérin_m_6
- removed link vérin_m_7
- removed link vérin_m_8
- removed link vérin_m_9
- added link base, mass 1e-9
- added link center, mass 139.99113879410862182; collision mesh filename=package:///center.stl; visual mesh filename=package:///center.stl
- added link cylinder_f, mass 2.7501984867936557499; collision mesh filename=package:///cylinder_f.stl; visual mesh filename=package:///cylinder_f.stl
- added link cylinder_f_10, mass 2.7501984867936557499; collision mesh filename=package:///cylinder_f.stl; visual mesh filename=package:///cylinder_f.stl
- added link cylinder_f_11, mass 2.7501984867936557499; collision mesh filename=package:///cylinder_f.stl; visual mesh filename=package:///cylinder_f.stl
- added link cylinder_f_12, mass 2.7501984867936557499; collision mesh filename=package:///cylinder_f.stl; visual mesh filename=package:///cylinder_f.stl
- added link cylinder_f_2, mass 2.7501984867936557499; collision mesh filename=package:///cylinder_f.stl; visual mesh filename=package:///cylinder_f.stl
- added link cylinder_f_3, mass 2.7501984867936557499; collision mesh filename=package:///cylinder_f.stl; visual mesh filename=package:///cylinder_f.stl
- added link cylinder_f_4, mass 2.7501984867936557499; collision mesh filename=package:///cylinder_f.stl; visual mesh filename=package:///cylinder_f.stl
- added link cylinder_f_5, mass 2.7501984867936557499; collision mesh filename=package:///cylinder_f.stl; visual mesh filename=package:///cylinder_f.stl
- added link cylinder_f_6, mass 2.7501984867936557499; collision mesh filename=package:///cylinder_f.stl; visual mesh filename=package:///cylinder_f.stl
- added link cylinder_f_7, mass 2.7501984867936557499; collision mesh filename=package:///cylinder_f.stl; visual mesh filename=package:///cylinder_f.stl
- added link cylinder_f_8, mass 2.7501984867936557499; collision mesh filename=package:///cylinder_f.stl; visual mesh filename=package:///cylinder_f.stl
- added link cylinder_f_9, mass 2.7501984867936557499; collision mesh filename=package:///cylinder_f.stl; visual mesh filename=package:///cylinder_f.stl
- added link cylinder_m, mass 2.7499900392833467322; collision mesh filename=package:///cylinder_m.stl; visual mesh filename=package:///cylinder_m.stl
- added link cylinder_m_10, mass 2.7499900392833467322; collision mesh filename=package:///cylinder_m.stl; visual mesh filename=package:///cylinder_m.stl
- added link cylinder_m_11, mass 2.7499900392833467322; collision mesh filename=package:///cylinder_m.stl; visual mesh filename=package:///cylinder_m.stl
- added link cylinder_m_12, mass 2.7499900392833467322; collision mesh filename=package:///cylinder_m.stl; visual mesh filename=package:///cylinder_m.stl
- added link cylinder_m_2, mass 2.7499900392833467322; collision mesh filename=package:///cylinder_m.stl; visual mesh filename=package:///cylinder_m.stl
- added link cylinder_m_3, mass 2.7499900392833467322; collision mesh filename=package:///cylinder_m.stl; visual mesh filename=package:///cylinder_m.stl
- added link cylinder_m_4, mass 2.7499900392833467322; collision mesh filename=package:///cylinder_m.stl; visual mesh filename=package:///cylinder_m.stl
- added link cylinder_m_5, mass 2.7499900392833467322; collision mesh filename=package:///cylinder_m.stl; visual mesh filename=package:///cylinder_m.stl
- added link cylinder_m_6, mass 2.7499900392833467322; collision mesh filename=package:///cylinder_m.stl; visual mesh filename=package:///cylinder_m.stl
- added link cylinder_m_7, mass 2.7499900392833467322; collision mesh filename=package:///cylinder_m.stl; visual mesh filename=package:///cylinder_m.stl
- added link cylinder_m_8, mass 2.7499900392833467322; collision mesh filename=package:///cylinder_m.stl; visual mesh filename=package:///cylinder_m.stl
- added link cylinder_m_9, mass 2.7499900392833467322; collision mesh filename=package:///cylinder_m.stl; visual mesh filename=package:///cylinder_m.stl
- added link cylinder_support, mass 3.4500000005941267034; collision mesh filename=package:///cylinder_support.stl; visual mesh filename=package:///cylinder_support.stl
- added link cylinder_support_2, mass 3.4500000005941267034; collision mesh filename=package:///cylinder_support.stl; visual mesh filename=package:///cylinder_support.stl
- added link cylinder_support_3, mass 3.4500000005941267034; collision mesh filename=package:///cylinder_support.stl; visual mesh filename=package:///cylinder_support.stl
- added link cylinder_support_4, mass 3.4500000005941267034; collision mesh filename=package:///cylinder_support.stl; visual mesh filename=package:///cylinder_support.stl
- added link femur, mass 3.599999998485739372; collision mesh filename=package:///femur.stl; visual mesh filename=package:///femur.stl
- added link femur_2, mass 3.599999998485739372; collision mesh filename=package:///femur.stl; visual mesh filename=package:///femur.stl
- added link femur_3, mass 3.599999998485739372; collision mesh filename=package:///femur.stl; visual mesh filename=package:///femur.stl
- added link femur_4, mass 3.599999998485739372; collision mesh filename=package:///femur.stl; visual mesh filename=package:///femur.stl
- added link foot, mass 3.649999995957899479; collision mesh filename=package:///foot.stl; visual mesh filename=package:///foot.stl
- added link foot_2, mass 3.649999995957899479; collision mesh filename=package:///foot.stl; visual mesh filename=package:///foot.stl
- added link foot_3, mass 3.649999995957899479; collision mesh filename=package:///foot.stl; visual mesh filename=package:///foot.stl
- added link foot_4, mass 3.649999995957899479; collision mesh filename=package:///foot.stl; visual mesh filename=package:///foot.stl
- added link hip, mass 3.599999992447649344; collision mesh filename=package:///hip.stl; visual mesh filename=package:///hip.stl
- added link hip_2, mass 3.599999992447649344; collision mesh filename=package:///hip.stl; visual mesh filename=package:///hip.stl
- added link hip_3, mass 3.599999992447649344; collision mesh filename=package:///hip.stl; visual mesh filename=package:///hip.stl
- added link hip_4, mass 3.599999992447649344; collision mesh filename=package:///hip.stl; visual mesh filename=package:///hip.stl
- added link l1_cl1_1, mass 1e-9
- added link l1_cl1_2, mass 1e-9
- added link l1_cl2_1, mass 1e-9
- added link l1_cl2_2, mass 1e-9
- added link l1_cl3_1, mass 1e-9
- added link l1_cl3_2, mass 1e-9
- added link l1_cl4_1, mass 1e-9
- added link l1_cl4_2, mass 1e-9
- added link l2_cl1_1, mass 1e-9
- added link l2_cl1_2, mass 1e-9
- added link l2_cl2_1, mass 1e-9
- added link l2_cl2_2, mass 1e-9
- added link l2_cl3_1, mass 1e-9
- added link l2_cl3_2, mass 1e-9
- added link l2_cl4_1, mass 1e-9
- added link l2_cl4_2, mass 1e-9
- added link l3_cl1_1, mass 1e-9
- added link l3_cl1_2, mass 1e-9
- added link l3_cl2_1, mass 1e-9
- added link l3_cl2_2, mass 1e-9
- added link l3_cl3_1, mass 1e-9
- added link l3_cl3_2, mass 1e-9
- added link l3_cl4_1, mass 1e-9
- added link l3_cl4_2, mass 1e-9
- added link l4_cl1_1, mass 1e-9
- added link l4_cl1_2, mass 1e-9
- added link l4_cl2_1, mass 1e-9
- added link l4_cl2_2, mass 1e-9
- added link l4_cl3_1, mass 1e-9
- added link l4_cl3_2, mass 1e-9
- added link l4_cl4_1, mass 1e-9
- added link l4_cl4_2, mass 1e-9
- added link leg_1, mass 1e-9
- added link leg_2, mass 1e-9
- added link leg_3, mass 1e-9
- added link leg_4, mass 1e-9
- link tibia: mass 3.57021 -> 3.999999995260936636; geometry collision mesh filename=package:///tibia.stl; visual mesh filename=package:///tibia.stl
- link tibia_2: mass 3.57021 -> 3.999999995260936636; geometry collision mesh filename=package:///tibia.stl; visual mesh filename=package:///tibia.stl
- link tibia_3: mass 3.57021 -> 3.999999995260936636; geometry collision mesh filename=package:///tibia.stl; visual mesh filename=package:///tibia.stl
- link tibia_4: mass 3.57021 -> 3.999999995260936636; geometry collision mesh filename=package:///tibia.stl; visual mesh filename=package:///tibia.stl
Joints:
- removed joint 00
- removed joint 01
- removed joint 02
- removed joint 03
- removed joint 04
- removed joint 05
- removed joint 06
- removed joint 07
- removed joint 0v1
- removed joint 0v2
- removed joint 0v3
- removed joint 10
- removed joint 11
- removed joint 12
- removed joint 13
- removed joint 14
- removed joint 15
- removed joint 16
- removed joint 17
- removed joint 1v1
- removed joint 1v2
- removed joint 1v3
- removed joint 20
- removed joint 21
- removed joint 22
- removed joint 23
- removed joint 24
- removed joint 25
- removed joint 26
- removed joint 27
- removed joint 2v1
- removed joint 2v2
- removed joint 2v3
- removed joint 30
- removed joint 31
- removed joint 32
- removed joint 33
- removed joint 34
- removed joint 35
- removed joint 36
- removed joint 37
- removed joint 3v1
- removed joint 3v2
- removed joint 3v3
- removed joint co_00
- removed joint co_01
- removed joint co_02
- removed joint co_03
- removed joint co_04
- removed joint co_05
- removed joint co_06
- removed joint co_07
- removed joint co_10
- removed joint co_11
- removed joint co_12
- removed joint co_13
- removed joint co_14
- removed joint co_15
- removed joint co_16
- removed joint co_17
- removed joint co_20
- removed joint co_21
- removed joint co_22
- removed joint co_23
- removed joint co_24
- removed joint co_25
- removed joint co_26
- removed joint co_27
- removed joint co_30
- removed joint co_31
- removed joint co_32
- removed joint co_33
- removed joint co_34
- removed joint co_35
- removed joint co_36
- removed joint co_37
- added joint base_frame: type fixed, parent center, child base, origin xyz=0 -0.52499999999999991118 0.025000000000000105471 rpy=0 -0 -1.570796326794896558, axis 0 0 0
- added joint l1_c1: type prismatic, parent cylinder_f, child cylinder_m, origin xyz=0.54016194822255925168 8.8817841970012523234e-16 1.7017248921313462451e-16 rpy=-1.3601114862349504746e-17 1.570796326794896336 0, axis 0 0 1, limit lower=0.036499999999999997724 upper=0.23649999999999998801 effort=1 velocity=20
- added joint l1_c2: type prismatic, parent cylinder_f_2, child cylinder_m_2, origin xyz=0.50159604710364502633 1.6653345369377348106e-15 -2.553512956637860043e-15 rpy=-1.4830109546207050645e-15 1.5707963267948930053 0, axis 0 0 1, limit lower=0.036499999999999997724 upper=0.23649999999999998801 effort=1 velocity=20
- added joint l1_c3: type prismatic, parent cylinder_f_3, child cylinder_m_3, origin xyz=0.55992619355683259652 1.5543122344752191566e-15 6.7168492989821970696e-15 rpy=3.1415926535897864547 -1.570796326794891673 0, axis 0 0 1, limit lower=0.036499999999999997724 upper=0.23649999999999998801 effort=1 velocity=20
- added joint l1_cl1_1_frame: type fixed, parent cylinder_m, child l1_cl1_1, origin xyz=0 0 -0.0095000000000000639488 rpy=-1.570796326794896558 -1.570796326794896558 0, axis 0 0 0
- added joint l1_cl1_2_frame: type fixed, parent hip, child l1_cl1_2, origin xyz=0.27500000000000013323 -5.5511151231257827021e-17 0.030000000000000002359 rpy=-1.570796326794896336 1.3210496169531149881e-16 -3.141592653589793116, axis 0 0 0
- added joint l1_cl2_1_frame: type fixed, parent cylinder_m_2, child l1_cl2_1, origin xyz=-4.4408920985006261617e-16 1.1102230246251565404e-16 -0.0094999999999998419042 rpy=-1.570796326794896558 -1.5707963267948958919 0, axis 0 0 0
- added joint l1_cl2_2_frame: type fixed, parent femur, child l1_cl2_2, origin xyz=-0.012999999999999789502 0.38400000000000000799 0.019999999999999795719 rpy=1.57079632679489678 7.2637879135570270462e-17 -6.7181087869012247853e-17, axis 0 0 0
- added joint l1_cl3_1_frame: type fixed, parent cylinder_m_3, child l1_cl3_1, origin xyz=1.1102230246251565404e-16 0 -0.0094999999999996198596 rpy=1.57079632679489678 1.570796326794896336 0, axis 0 0 0
- added joint l1_cl3_2_frame: type fixed, parent foot, child l1_cl3_2, origin xyz=-2.2204460492503130808e-16 -0.50500000000000011546 0.020000000000000184297 rpy=-1.570796326794896558 5.9381623995301617414e-16 3.141592653589793116, axis 0 0 0
- added joint l1_cl4_1_frame: type fixed, parent cylinder_support, child l1_cl4_1, origin xyz=0 0.58999999999999996891 0.019999999999999573674 rpy=1.5707963267948936714 -3.6993336504632930902e-17 -3.141592653589793116, axis 0 0 0
- added joint l1_cl4_2_frame: type fixed, parent tibia, child l1_cl4_2, origin xyz=-0.44999999999999995559 0 -0.020000000000000184297 rpy=-1.570796326794896558 6.5422720734645307412e-18 -3.141592653589793116, axis 0 0 0
- added joint l1_r1: type revolute, parent center, child cylinder_f, origin xyz=-0.44000000000000016875 -0.33500000000000024203 1.0755285551056207683e-16 rpy=3.1415926535897922278 -2.3595482621880709577e-16 -1.2888338553123910302, axis 0 0 1, limit lower=0 upper=1.570796326794896558 effort=1 velocity=20
- added joint l1_r2: type revolute, parent center, child hip, origin xyz=-0.50000000000000011102 -1.0250000000000001332 0.030000000000000102973 rpy=3.141592653589793116 -3.0599760784490747333e-18 0.71499248882173183084, axis 0 0 1, limit lower=0 upper=1.570796326794896558 effort=1 velocity=20
- added joint l1_r3: type revolute, parent hip, child femur, origin xyz=0.12500000000000022204 -0.019999999999999906741 -0.040000000000000007772 rpy=-1.570796326794896558 0.35430516897438335544 8.333430058132758542e-15, axis 0 0 1, limit lower=-1.570796326794896558 upper=1.570796326794896558 effort=1 velocity=20
- added joint l1_r4: type revolute, parent femur, child tibia, origin xyz=-1.1102230246251565404e-16 0.48999999999999999112 -2.2204460492503130808e-16 rpy=3.1415926535897900074 2.7294237846170472709e-15 -0.35430516897438252277, axis 0 0 1, limit lower=-1.570796326794896558 upper=1.570796326794896558 effort=1 velocity=20
- added joint l1_r5: type revolute, parent tibia, child foot, origin xyz=-0.75 -1.1102230246251565404e-16 -0.040000000000000146549 rpy=-5.6175769265896188431e-16 1.3875289317899453937e-15 3.141592653589793116, axis 0 0 1, limit lower=-1.570796326794896558 upper=1.570796326794896558 effort=1 velocity=20
- added joint l1_r6: type revolute, parent hip, child cylinder_f_2, origin xyz=-0.40999999999999992006 1.6653345369377348106e-16 -0.094999999999999987232 rpy=1.570796326794896558 0.65724109672367558854 -6.6514940932233617718e-15, axis 0 0 1, limit lower=0 upper=1.570796326794896558 effort=1 velocity=20
- added joint l1_r7: type revolute, parent hip, child cylinder_support, origin xyz=-0.12499999999999822364 -0.020000000000001849632 -0.040000000000000007772 rpy=-1.570796326794896558 0.67784852797306960337 -1.2527273977519951284e-15, axis 0 0 1, limit lower=-1.570796326794896558 upper=1.570796326794896558 effort=1 velocity=20
- added joint l1_r8: type revolute, parent cylinder_support, child cylinder_f_3, origin xyz=2.2204460492503130808e-16 0.39249999999999996003 0.020000000000001461054 rpy=6.6758930342687408726e-15 1.8103960944874226249e-14 -3.1275650633842229098, axis 0 0 1, limit lower=0 upper=1.570796326794896558 effort=1 velocity=20
- added joint l2_c1: type prismatic, parent cylinder_f_4, child cylinder_m_4, origin xyz=0.54016194822256369257 -3.6082248300317587564e-16 9.9643341442874709379e-17 rpy=1.7558505235703240888e-16 1.5707963267948950037 0, axis 0 0 1, limit lower=0.036499999999999997724 upper=0.23649999999999998801 effort=1 velocity=20
- added joint l2_c2: type prismatic, parent cylinder_f_5, child cylinder_m_5, origin xyz=0.50159604710360994329 0 1.4988010832439613296e-15 rpy=1.072854554705450715e-16 1.5707963267948927832 0, axis 0 0 1, limit lower=0.036499999999999997724 upper=0.23649999999999998801 effort=1 velocity=20
- added joint l2_c3: type prismatic, parent cylinder_f_6, child cylinder_m_6, origin xyz=0.55992619355683270754 -2.4424906541753443889e-15 5.1070259132757200859e-15 rpy=3.1415926535897789051 -1.5707963267948827912 0, axis 0 0 1, limit lower=0.036499999999999997724 upper=0.23649999999999998801 effort=1 velocity=20
- added joint l2_cl1_1_frame: type fixed, parent cylinder_m_4, child l2_cl1_1, origin xyz=9.8607613152626475676e-32 0 -0.0095000000000000639488 rpy=-1.5707963267948970021 -1.5707963267948954478 0, axis 0 0 0
- added joint l2_cl1_2_frame: type fixed, parent hip_2, child l2_cl1_2, origin xyz=0.2750000000000000222 5.5511151231257827021e-17 0.02999999999999999889 rpy=-1.570796326794896336 5.8999261890123604462e-17 -3.1415926535897926719, axis 0 0 0
- added joint l2_cl2_1_frame: type fixed, parent cylinder_m_5, child l2_cl2_1, origin xyz=5.5511151231257827021e-17 -1.1102230246251565404e-16 -0.0094999999999999962946 rpy=-1.570796326794896558 -1.5707963267948930053 0, axis 0 0 0
- added joint l2_cl2_2_frame: type fixed, parent femur_2, child l2_cl2_2, origin xyz=-0.013000000000000011546 0.38400000000000000799 0.020000000000000073275 rpy=1.570796326794896558 -2.9099399159039228985e-16 -7.2338255418286372255e-17, axis 0 0 0
- added joint l2_cl3_1_frame: type fixed, parent cylinder_m_6, child l2_cl3_1, origin xyz=1.6653345369377348106e-16 0 -0.0095000000000000639488 rpy=1.570796326794896558 1.5707963267948956698 0, axis 0 0 0
- added joint l2_cl3_2_frame: type fixed, parent foot_2, child l2_cl3_2, origin xyz=0 -0.50500000000000000444 0.020000000000000017764 rpy=-1.570796326794896558 -8.5901255498107134466e-16 -3.141592653589793116, axis 0 0 0
- added joint l2_cl4_1_frame: type fixed, parent cylinder_support_2, child l2_cl4_1, origin xyz=0 0.58999999999999996891 0.020000000000000184297 rpy=1.5707963267948941155 -6.8893610029579801103e-15 -3.141592653589793116, axis 0 0 0
- added joint l2_cl4_2_frame: type fixed, parent tibia_2, child l2_cl4_2, origin xyz=-0.44999999999999990008 0 -0.01999999999999985123 rpy=-1.570796326794896558 2.0671484703801979509e-17 3.141592653589793116, axis 0 0 0
- added joint l2_r1: type revolute, parent center, child cylinder_f_4, origin xyz=0.18999999999999972466 -0.08499999999999972855 1.0755285551056199055e-16 rpy=3.141592653589793116 -1.6993414331267333812e-16 -2.8596301821072906968, axis 0 0 1, limit lower=0 upper=1.570796326794896558 effort=1 velocity=20
- added joint l2_r2: type revolute, parent center, child hip_2, origin xyz=-0.50000000000000011102 -0.024999999999999852202 0.030000000000000096034 rpy=3.141592653589793116 -1.1535304933115970508e-16 -0.85580383797315651151, axis 0 0 1, limit lower=0 upper=1.570796326794896558 effort=1 velocity=20
- added joint l2_r3: type revolute, parent hip_2, child femur_2, origin xyz=0.12500000000000011102 -0.02000000000000035083 -0.040000000000000028588 rpy=-1.570796326794896336 0.35430516897447805746 -2.2175415972529100751e-15, axis 0 0 1, limit lower=-1.570796326794896558 upper=1.570796326794896558 effort=1 velocity=20
- added joint l2_r4: type revolute, parent femur_2, child tibia_2, origin xyz=1.6653345369377348106e-16 0.48999999999999965805 -4.4408920985006261617e-16 rpy=3.141592653589793116 -3.4782139178269834916e-15 -0.35430516897447428271, axis 0 0 1, limit lower=-1.570796326794896558 upper=1.570796326794896558 effort=1 velocity=20
- added joint l2_r5: type revolute, parent tibia_2, child foot_2, origin xyz=-0.75 -1.1102230246251565404e-16 -0.039999999999999980016 rpy=-9.4612926646945399132e-16 1.9371594980863719444e-16 -3.141592653589793116, axis 0 0 1, limit lower=-1.570796326794896558 upper=1.570796326794896558 effort=1 velocity=20
- added joint l2_r6: type revolute, parent hip_2, child cylinder_f_5, origin xyz=-0.40999999999999980904 7.2164496600635175128e-16 -0.095000000000000028866 rpy=1.570796326794896558 0.65724109672367858614 -5.1466463596763776877e-15, axis 0 0 1, limit lower=0 upper=1.570796326794896558 effort=1 velocity=20
- added joint l2_r7: type revolute, parent hip_2, child cylinder_support_2, origin xyz=-0.1249999999999990008 -0.019999999999999074074 -0.040000000000000000833 rpy=-1.570796326794896558 0.67784852797311845318 6.530241321319161551e-15, axis 0 0 1, limit lower=-1.570796326794896558 upper=1.570796326794896558 effort=1 velocity=20
- added joint l2_r8: type revolute, parent cylinder_support_2, child cylinder_f_6, origin xyz=2.2204460492503130808e-16 0.39249999999999984901 0.01999999999999985123 rpy=6.0491518543493472829e-15 3.6588336647256622468e-15 -3.1275650633842677628, axis 0 0 1, limit lower=0 upper=1.570796326794896558 effort=1 velocity=20
- added joint l3_c1: type prismatic, parent cylinder_f_7, child cylinder_m_7, origin xyz=0.54016194822258023489 3.1086244689504383132e-15 -9.140831766129502433e-16 rpy=-1.8325883609705074827e-16 1.5707963267948930053 0, axis 0 0 1, limit lower=0.036499999999999997724 upper=0.23649999999999998801 effort=1 velocity=20
- added joint l3_c2: type prismatic, parent cylinder_f_8, child cylinder_m_8, origin xyz=0.5015960471036677859 -4.4408920985006261617e-16 2.2204460492503130808e-16 rpy=-6.354613258499769017e-17 1.5707963267948921171 0, axis 0 0 1, limit lower=0.036499999999999997724 upper=0.23649999999999998801 effort=1 velocity=20
- added joint l3_c3: type prismatic, parent cylinder_f_9, child cylinder_m_9, origin xyz=0.55992619355682637927 -3.5527136788005009294e-15 -2.2204460492503130808e-15 rpy=-3.141592653589793116 -1.570796326794896336 0, axis 0 0 1, limit lower=0.036499999999999997724 upper=0.23649999999999998801 effort=1 velocity=20
- added joint l3_cl1_1_frame: type fixed, parent cylinder_m_7, child l3_cl1_1, origin xyz=0 2.7755575615628913511e-17 -0.0095000000000000084377 rpy=-1.570796326794896558 -1.570796326794896558 0, axis 0 0 0
- added joint l3_cl1_2_frame: type fixed, parent hip_3, child l3_cl1_2, origin xyz=0.27499999999999980016 0 0.02999999999999999889 rpy=-1.570796326794896558 -4.4969093478228596159e-29 3.1415926535897922278, axis 0 0 0
- added joint l3_cl2_1_frame: type fixed, parent cylinder_m_8, child l3_cl2_1, origin xyz=-5.5511151231257827021e-17 0 -0.0094999999999999668043 rpy=-1.5707963267948972241 -1.570796326794896336 0, axis 0 0 0
- added joint l3_cl2_2_frame: type fixed, parent femur_3, child l3_cl2_2, origin xyz=-0.013000000000000067057 0.3840000000000000635 0.020000000000000017764 rpy=1.570796326794896558 -5.2424180237022428121e-16 -6.8688372249162086865e-17, axis 0 0 0
- added joint l3_cl3_1_frame: type fixed, parent cylinder_m_9, child l3_cl3_1, origin xyz=-1.1102230246251565404e-16 0 -0.0094999999999997308819 rpy=1.57079632679489678 1.570796326794896336 0, axis 0 0 0
- added joint l3_cl3_2_frame: type fixed, parent foot_3, child l3_cl3_2, origin xyz=0 -0.50499999999999989342 0.020000000000000073275 rpy=-1.570796326794896558 3.5164344829539952788e-16 3.1415926535897926719, axis 0 0 0
- added joint l3_cl4_1_frame: type fixed, parent cylinder_support_3, child l3_cl4_1, origin xyz=-1.6653345369377348106e-16 0.59000000000000007994 0.019999999999999962252 rpy=1.570796326794896558 -9.0419128252829653613e-17 3.141592653589793116, axis 0 0 0
- added joint l3_cl4_2_frame: type fixed, parent tibia_3, child l3_cl4_2, origin xyz=-0.45000000000000012212 -1.1102230246251565404e-16 -0.019999999999999906741 rpy=-1.570796326794896558 -7.1621134632402218173e-17 3.141592653589793116, axis 0 0 0
- added joint l3_r1: type revolute, parent center, child cylinder_f_7, origin xyz=0.44000000000000055733 -0.71499999999999974687 1.0755285551056202753e-16 rpy=-3.1415926535897904515 3.2403040233095439527e-24 1.8527587982774034181, axis 0 0 1, limit lower=0 upper=1.570796326794896558 effort=1 velocity=20
- added joint l3_r2: type revolute, parent center, child hip_3, origin xyz=0.49999999999999994449 -0.024999999999999918121 0.030000000000000102973 rpy=-3.1415926535897922278 -8.7006547959070078248e-16 -2.4266001647680677245, axis 0 0 1, limit lower=0 upper=1.570796326794896558 effort=1 velocity=20
- added joint l3_r3: type revolute, parent hip_3, child femur_3, origin xyz=0.12499999999999980571 -0.019999999999999962252 -0.04000000000000001471 rpy=-1.57079632679489678 0.35430516897432023926 6.1122737486658637803e-15, axis 0 0 1, limit lower=-1.570796326794896558 upper=1.570796326794896558 effort=1 velocity=20
- added joint l3_r4: type revolute, parent femur_3, child tibia_3, origin xyz=-2.7755575615628913511e-17 0.49000000000000004663 -5.5511151231257827021e-17 rpy=3.1415926535897873428 2.9877259684137084701e-15 -0.35430516897432418055, axis 0 0 1, limit lower=-1.570796326794896558 upper=1.570796326794896558 effort=1 velocity=20
- added joint l3_r5: type revolute, parent tibia_3, child foot_3, origin xyz=-0.75000000000000022204 0 -0.03999999999999970246 rpy=-1.1255613980499141844e-15 -3.2685853399614706325e-15 -3.141592653589793116, axis 0 0 1, limit lower=-1.570796326794896558 upper=1.570796326794896558 effort=1 velocity=20
- added joint l3_r6: type revolute, parent hip_3, child cylinder_f_8, origin xyz=-0.4100000000000000866 4.9960036108132044319e-16 -0.095000000000000056621 rpy=1.5707963267948994446 0.65724109672367359014 1.8096855595557680072e-15, axis 0 0 1, limit lower=0 upper=1.570796326794896558 effort=1 velocity=20
- added joint l3_r7: type revolute, parent hip_3, child cylinder_support_3, origin xyz=-0.12500000000000011102 -0.019999999999999795719 -0.039999999999999986955 rpy=-1.57079632679489678 0.67784852797300643168 -3.8844866652341196646e-15, axis 0 0 1, limit lower=-1.570796326794896558 upper=1.570796326794896558 effort=1 velocity=20
- added joint l3_r8: type revolute, parent cylinder_support_3, child cylinder_f_9, origin xyz=-5.5511151231257827021e-17 0.39250000000000023759 0.019999999999999962252 rpy=-1.4752362061541671842e-15 -1.1273800577279551433e-15 -3.1275650633841585169, axis 0 0 1, limit lower=0 upper=1.570796326794896558 effort=1 velocity=20
- added joint l4_c1: type prismatic, parent cylinder_f_10, child cylinder_m_10, origin xyz=0.54016194822257568298 -1.1102230246251565404e-16 3.2215294379649110445e-16 rpy=1.9525057998941007146e-16 1.5707963267948952257 0, axis 0 0 1, limit lower=0.036499999999999997724 upper=0.23649999999999998801 effort=1 velocity=20
- added joint l4_c2: type prismatic, parent cylinder_f_11, child cylinder_m_11, origin xyz=0.5015960471036094992 -1.1102230246251565404e-15 -1.9984014443252817728e-15 rpy=-1.4206229417985893165e-15 1.5707963267948938935 0, axis 0 0 1, limit lower=0.036499999999999997724 upper=0.23649999999999998801 effort=1 velocity=20
- added joint l4_c3: type prismatic, parent cylinder_f_12, child cylinder_m_12, origin xyz=0.55992619355684736249 -3.7747582837255322374e-15 4.8294701571194309508e-15 rpy=3.1415926535897864547 -1.5707963267948921171 0, axis 0 0 1, limit lower=0.036499999999999997724 upper=0.23649999999999998801 effort=1 velocity=20
- added joint l4_cl1_1_frame: type fixed, parent cylinder_m_10, child l4_cl1_1, origin xyz=0 0 -0.0094999999999999668043 rpy=-1.570796326794896558 -1.570796326794896336 0, axis 0 0 0
- added joint l4_cl1_2_frame: type fixed, parent hip_4, child l4_cl1_2, origin xyz=0.2750000000000000222 1.1102230246251565404e-16 0.029999999999999991951 rpy=-1.5707963267948956698 5.5104333540991556298e-16 -3.1415926535897926719, axis 0 0 0
- added joint l4_cl2_1_frame: type fixed, parent cylinder_m_11, child l4_cl2_1, origin xyz=5.5511151231257827021e-17 0 -0.0094999999999996198596 rpy=-1.57079632679489678 -1.5707963267948958919 0, axis 0 0 0
- added joint l4_cl2_2_frame: type fixed, parent femur_4, child l4_cl2_2, origin xyz=-0.012999999999999678479 0.3840000000000000635 0.019999999999999795719 rpy=1.570796326794896558 -4.8590027552132278873e-16 -2.6823769382526587703e-16, axis 0 0 0
- added joint l4_cl3_1_frame: type fixed, parent cylinder_m_12, child l4_cl3_1, origin xyz=-2.2204460492503130808e-16 -2.2204460492503130808e-16 -0.0094999999999996198596 rpy=1.570796326794896558 1.5707963267948952257 0, axis 0 0 0
- added joint l4_cl3_2_frame: type fixed, parent foot_4, child l4_cl3_2, origin xyz=0 -0.50500000000000011546 0.020000000000000295319 rpy=-1.570796326794896558 1.0095225613817616779e-15 -3.141592653589793116, axis 0 0 0
- added joint l4_cl4_1_frame: type fixed, parent cylinder_support_4, child l4_cl4_1, origin xyz=-1.1102230246251565404e-16 0.59000000000000030198 0.01999999999999985123 rpy=1.57079632679489678 -7.2679738829527707955e-16 3.1415926535897917837, axis 0 0 0
- added joint l4_cl4_2_frame: type fixed, parent tibia_4, child l4_cl4_2, origin xyz=-0.45000000000000039968 0 -0.020000000000000073275 rpy=-1.570796326794896558 1.2508912073766756774e-16 -3.141592653589793116, axis 0 0 0
- added joint l4_r1: type revolute, parent center, child cylinder_f_10, origin xyz=-0.18999999999999961364 -0.96499999999999985789 1.0755285551056070865e-16 rpy=3.1415926535897908956 1.9044041489550536811e-24 0.28196247148250824788, axis 0 0 1, limit lower=0 upper=1.570796326794896558 effort=1 velocity=20
- added joint l4_r2: type revolute, parent center, child hip_4, origin xyz=0.5 -1.0249999999999999112 0.030000000000000099504 rpy=-3.1415926535897926719 7.8766131130756764154e-16 2.2857888156166228377, axis 0 0 1, limit lower=0 upper=1.570796326794896558 effort=1 velocity=20
- added joint l4_r3: type revolute, parent hip_4, child femur_4, origin xyz=0.12500000000000732747 -0.019999999999993856026 -0.039999999999999896749 rpy=-1.5707963267948958919 0.35430516897449731983 1.1506556893667557454e-14, axis 0 0 1, limit lower=-1.570796326794896558 upper=1.570796326794896558 effort=1 velocity=20
- added joint l4_r4: type revolute, parent femur_4, child tibia_4, origin xyz=1.1102230246251565404e-15 0.48999999999999860334 2.0539125955565395998e-15 rpy=3.1415926535897895633 4.8455040699935128072e-15 -0.35430516897449099156, axis 0 0 1, limit lower=-1.570796326794896558 upper=1.570796326794896558 effort=1 velocity=20
- added joint l4_r5: type revolute, parent tibia_4, child foot_4, origin xyz=-0.75 3.3306690738754696213e-16 -0.040000000000000035527 rpy=-6.4405352938840367248e-15 8.4157945655509966573e-15 -3.141592653589793116, axis 0 0 1, limit lower=-1.570796326794896558 upper=1.570796326794896558 effort=1 velocity=20
- added joint l4_r6: type revolute, parent hip_4, child cylinder_f_11, origin xyz=-0.40999999999999836575 1.4988010832439613296e-15 -0.094999999999999917843 rpy=1.5707963267949027752 0.65724109672369257495 3.5697696165855604194e-15, axis 0 0 1, limit lower=0 upper=1.570796326794896558 effort=1 velocity=20
- added joint l4_r7: type revolute, parent hip_4, child cylinder_support_4, origin xyz=-0.12500000000000133227 -0.019999999999999684697 -0.03999999999999995226 rpy=-1.5707963267949001107 0.67784852797314421036 -1.4595506346581353191e-14, axis 0 0 1, limit lower=-1.570796326794896558 upper=1.570796326794896558 effort=1 velocity=20
- added joint l4_r8: type revolute, parent cylinder_support_4, child cylinder_f_12, origin xyz=0 0.3925000000000002931 0.019999999999999573674 rpy=3.5707879082592744506e-15 2.3225679053517195645e-14 -3.127565063384278865, axis 0 0 1, limit lower=0 upper=1.570796326794896558 effort=1 velocity=20
- added joint leg_1_frame: type fixed, parent foot, child leg_1, origin xyz=0.004999999999999671374 -1.0075000000000000622 0.020000000000000239808 rpy=-1.570796326794896558 -3.7290365520547414402e-16 -1.4139732311379854492e-28, axis 0 0 0
- added joint leg_2_frame: type fixed, parent foot_2, child leg_2, origin xyz=0.0049999999999998934186 -1.0074999999999998401 0.020000000000000184297 rpy=-1.570796326794896558 2.1015511443037622533e-16 -5.1910748321200000537e-18, axis 0 0 0
- added joint leg_3_frame: type fixed, parent foot_3, child leg_3, origin xyz=0.0049999999999998934186 -1.0074999999999998401 0.020000000000000017764 rpy=-1.570796326794896558 -1.0354129802097694568e-16 -6.2450045135172953869e-16, axis 0 0 0
- added joint leg_4_frame: type fixed, parent foot_4, child leg_4, origin xyz=0.0050000000000001154632 -1.0075000000000000622 0.020000000000000073275 rpy=-1.570796326794896558 -8.3307679057966979047e-16 8.3266726846905118526e-17, axis 0 0 0
